File: PCB/MIDI-harmonica.kicad_pcb (KiCad board)
At the start: 2 copper layers, 96 x 47.5 mm, 17 parts, among them J1 Screw_Terminal_01x02, SW1 SW_SP3T, SW2 SW_Push, SW3 SW_Push, U0 XIAO-ESP32-S3-Plus-SMD

Commit message: update
Routing:
- net /U10: track 82.5 -> 81.0 mm
Changed lines of the file:
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@@
 		(at 135.5 108)
 		(property "Reference" "JS1"
-			(at -6 -10 0)
+			(at 0 1 0)
 			(unlocked yes)
 			(layer "F.SilkS")
@@
 		(at 145 99)
 		(property "Reference" "SW1"
-			(at 8.5 -1 0)
+			(at 1.5 2 0)
 			(unlocked yes)
 			(layer "F.SilkS")
@@
 	)
 	(segment
-		(start 164.338478 100.5)
-		(end 169.161522 100.5)
-		(width 0.2)
-		(layer "B.Cu")
-		(net "/U10")
-	)
-	(segment
-		(start 162.961522 100.8)
-		(end 164.038478 100.8)
-		(width 0.2)
-		(layer "B.Cu")
-		(net "/U10")
-	)
-	(segment
-		(start 169.461522 100.8)
-		(end 170.538478 100.8)
-		(width 0.2)
-		(layer "B.Cu")
-		(net "/U10")
-	)
-	(segment
-		(start 164.038478 100.8)
-		(end 164.338478 100.5)
-		(width 0.2)
-		(layer "B.Cu")
-		(net "/U10")
-	)
-	(segment
-		(start 150.585786 100.4)
-		(end 151.414214 100.4)
-		(width 0.2)
-		(layer "B.Cu")
-		(net "/U10")
-	)
-	(segment
-		(start 176.161522 100.5)
-		(end 176.461522 100.8)
-		(width 0.2)
-		(layer "B.Cu")
-		(net "/U10")
-	)
-	(segment
-		(start 169.161522 100.5)
-		(end 169.461522 100.8)
-		(width 0.2)
-		(layer "B.Cu")
-		(net "/U10")
-	)
-	(segment
-		(start 139.414214 100.4)
-		(end 139.814214 100)
+		(start 127 100)
+		(end 138.185786 100)
 		(width 0.2)
 		(layer "B.Cu")
@@
 	(segment
 		(start 138.185786 100)
-		(end 138.585786 100.4)
+		(end 139.185787 101)
 		(width 0.2)
 		(layer "B.Cu")
@@
 	)
 	(segment
-		(start 151.814214 100)
-		(end 162.161522 100)
-		(width 0.2)
-		(layer "B.Cu")
-		(net "/U10")
-	)
-	(segment
-		(start 177.838478 100.5)
-		(end 179 100.5)
-		(width 0.2)
-		(layer "B.Cu")
-		(net "/U10")
-	)
-	(segment
-		(start 179 100.5)
-		(end 180 101.5)
-		(width 0.2)
-		(layer "B.Cu")
-		(net "/U10")
-	)
-	(segment
-		(start 170.538478 100.8)
-		(end 170.838478 100.5)
-		(width 0.2)
-		(layer "B.Cu")
-		(net "/U10")
-	)
-	(segment
-		(start 150.185786 100)
-		(end 150.585786 100.4)
-		(width 0.2)
-		(layer "B.Cu")
-		(net "/U10")
-	)
-	(segment
-		(start 177.538478 100.8)
-		(end 177.838478 100.5)
-		(width 0.2)
-		(layer "B.Cu")
-		(net "/U10")
-	)
-	(segment
-		(start 139.814214 100)
-		(end 150.185786 100)
+		(start 139.185787 101)
+		(end 179.5 101)
 		(width 0.2)
 		(layer "B.Cu")
@@
 	)
 	(segment
-		(start 170.838478 100.5)
-		(end 176.161522 100.5)
+		(start 179.5 101)
+		(end 180 101.5)
 		(width 0.2)
 		(layer "B.Cu")
@@
 	)
 	(segment
-		(start 162.161522 100)
-		(end 162.961522 100.8)
-		(width 0.2)
-		(layer "B.Cu")
-		(net "/U10")
-	)
-	(segment
-		(start 138.585786 100.4)
-		(end 139.414214 100.4)
-		(width 0.2)
-		(layer "B.Cu")
-		(net "/U10")
-	)
-	(segment
-		(start 151.414214 100.4)
-		(end 151.814214 100)
-		(width 0.2)
-		(layer "B.Cu")
-		(net "/U10")
-	)
-	(segment
-		(start 127 100)
-		(end 138.185786 100)
-		(width 0.2)
-		(layer "B.Cu")
-		(net "/U10")
-	)
-	(segment
-		(start 176.461522 100.8)
-		(end 177.538478 100.8)
-		(width 0.2)
-		(layer "B.Cu")
-		(net "/U10")
-	)
-	(segment
 		(start 107.145686 103.58)
 		(end 123.665686 120.1)
@@
 		(net "/U8")
 	)
-	(segment
-		(start 165 102.225)
-		(end 166.254365 102.225)
-		(width 0.2)
-		(layer "F.Cu")
-		(net "/U8")
-	)
 	(via
 		(at 168.529365 104.5)
@@
 	)
 	(via
-		(at 165 102.225)
+		(at 166.254365 102.225)
 		(size 0.6)
 		(drill 0.3)
@@
 	)
 	(segment
-		(start 139.579899 100.8)
-		(end 138.4201 100.8)
-		(width 0.2)
-		(layer "B.Cu")
-		(net "/U8")
-	)
-	(segment
-		(start 138.4201 100.8)
-		(end 138.1201 100.5)
-		(width 0.2)
-		(layer "B.Cu")
-		(net "/U8")
-	)
-	(segment
-		(start 125.71 100.5)
-		(end 123.9 102.31)
-		(width 0.2)
-		(layer "B.Cu")
-		(net "/U8")
-	)
-	(segment
-		(start 151.8799 100.5)
-		(end 151.579899 100.8)
-		(width 0.2)
-		(layer "B.Cu")
-		(net "/U8")
-	)
-	(segment
-		(start 162.795836 101.2)
-		(end 162.095836 100.5)
+		(start 166.254365 102.225)
+		(end 166.029365 102)
 		(width 0.2)
 		(layer "B.Cu")
@@
 	)
 	(segment
-		(start 162.095836 100.5)
-		(end 151.8799 100.5)
-		(width 0.2)
-		(layer "B.Cu")
-		(net "/U8")
-	)
-	(segment
-		(start 150.4201 100.8)
-		(end 150.1201 100.5)
-		(width 0.2)
-		(layer "B.Cu")
-		(net "/U8")
-	)
-	(segment
-		(start 139.8799 100.5)
-		(end 139.579899 100.8)
-		(width 0.2)
-		(layer "B.Cu")
-		(net "/U8")
-	)
-	(segment
-		(start 163.975 101.2)
-		(end 162.795836 101.2)
-		(width 0.2)
-		(layer "B.Cu")
-		(net "/U8")
-	)
-	(segment
-		(start 150.1201 100.5)
-		(end 139.8799 100.5)
+		(start 139.6201 102)
+		(end 138.1201 100.5)
 		(width 0.2)
 		(layer "B.Cu")
@@
 	)
 	(segment
-		(start 165 102.225)
-		(end 163.975 101.2)
+		(start 166.029365 102)
+		(end 139.6201 102)
 		(width 0.2)
 		(layer "B.Cu")
@@
 	)
 	(segment
-		(start 151.579899 100.8)
-		(end 150.4201 100.8)
+		(start 125.71 100.5)
+		(end 123.9 102.31)
 		(width 0.2)
 		(layer "B.Cu")
